Commit message: Trying simulation with just the aquatic part.

File: haubentaucher_description/urdf/haubentaucher_multirotor_base.xacro (robot description, xacro)
@@ -17,4 +17,44 @@
 -->
 <robot xmlns:xacro="http://ros.org/wiki/xacro">
+  <!--
+  Center of buoyancy according to eq. (3.1) p. 28 in Berg2012.
+  The original values, [0.0822, -0.00773, 0.3872] however, seem to
+  assume NWU (otherwise cob is below cog?).
+  -->
+  <xacro:property name="cob" value="0.0 0.0 0.3"/>
+  <!-- Volume, see p.31 in Berg2012 -->
+  <xacro:property name="volume" value="0.83826"/>
+  <xacro:macro name="rexrov_hydro_model" params="namespace">
+      <link name="${namespace}/base_link_inertia">
+          <neutrally_buoyant>1</neutrally_buoyant>
+          <volume>${volume}</volume>
+          <box>
+              <width>1.5</width>
+              <length>2.6</length>
+              <height>1.6</height>
+          </box>
+          <center_of_buoyancy>${cob}</center_of_buoyancy>
+          <hydrodynamic_model>
+              <type>fossen</type>
+              <!-- Added mass: see p.28 in Berg2012 -->
+              <added_mass>
+                   779.79 -6.8773 -103.32  8.5426 -165.54 -7.8033
+                  -6.8773    1222   51.29  409.44 -5.8488  62.726
+                  -103.32   51.29  3659.9  6.1112 -386.42  10.774
+                   8.5426  409.44  6.1112   534.9 -10.027  21.019
+                  -165.54 -5.8488 -386.42 -10.027  842.69 -1.1162
+                  -7.8033  62.726  10.775  21.019 -1.1162  224.32
+              </added_mass>
+              <!-- Linear damping: see p.31 in Berg2012 -->
+              <linear_damping>
+                  -74.82 -69.48 -728.4 -268.8 -309.77 -105
+              </linear_damping>
+              <!-- Non-linear damping: see p.30 in Berg2012 -->
+              <quadratic_damping>
+                  -748.22 -992.53 -1821.01 -672 -774.44 -523.27
+              </quadratic_damping>
+          </hydrodynamic_model>
+      </link>
+  </xacro:macro>
   <!-- Macro for the inertia of a box -->
   <xacro:macro name="box_inertia" params="x y z mass">
@@ -72,4 +112,13 @@
         <linkName>${robot_namespace}/base_link</linkName>
         <rotorVelocitySlowdownSim>${rotor_velocity_slowdown_sim}</rotorVelocitySlowdownSim>
+      </plugin>
+    </gazebo>
+    <gazebo>
+      <plugin name="uuv_plugin" filename="libuuv_underwater_object_ros_plugin.so">
+        <fluid_density>1028.0</fluid_density>
+        <flow_velocity_topic>hydrodynamics/current_velocity</flow_velocity_topic>
+        <debug>True</debug>
+        <!-- Adding the hydrodynamic and hydrostatic parameters for the vehicle-->
+        <xacro:rexrov_hydro_model namespace="${robot_namespace}"/>
       </plugin>
     </gazebo>
