Commit message: added blades

File: haubentaucher_description/urdf/rexrov_actuators.xacro (robot description, xacro)
@@ -13,5 +13,5 @@
 -->
 <robot xmlns:xacro="http://www.ros.org/wiki/xacro">
-  <xacro:property name="prop_mesh_file" value="file://$(find uuv_descriptions)/meshes/prop.dae"/>
+  <xacro:property name="prop_mesh_file" value="file://$(find haubentaucher_description)/meshes/prop.stl"/>
   <!-- Thruster joint and link snippet -->
   <xacro:macro name="thruster_macro"
@@ -27,5 +27,11 @@
   </xacro:macro>
   <xacro:thruster_macro namespace="${namespace}" thruster_id="0">
-    <origin xyz="-0.890895 0.334385 0.528822" rpy="${0*d2r} ${-74.53*d2r} ${-53.21*d2r}"/>
+    <origin xyz="0.12 0 0" rpy="0 0 0"/>
+  </xacro:thruster_macro>
+  <xacro:thruster_macro namespace="${namespace}" thruster_id="1">
+    <origin xyz="0 -0.3 0" rpy="0 0 0"/>
+  </xacro:thruster_macro>
+  <xacro:thruster_macro namespace="${namespace}" thruster_id="2">
+    <origin xyz="0 0.3 0" rpy="0 0 0"/>
   </xacro:thruster_macro>
 </robot>

File: haubentaucher_description/urdf/rexrov_base.xacro (robot description, xacro)
@@ -49,7 +49,7 @@
       <!-- bottom plate -->
       <collision>
-        <origin xyz="0 0 0" rpy="0 0 0" />
+        <origin xyz="0 0 0" rpy="0 0 0"/>
         <geometry>
-          <box size="${body_width} ${body_width} ${body_height}"/> <!-- [m] [m] [m] -->
+          <mesh filename="${visual_mesh_file}" scale="1 1 1"/>
         </geometry>
       </collision>
