Commit message: trying some values to added mass.

File: haubentaucher_description/urdf/rexrov.gazebo.xacro (robot description, xacro)
@@ -18,7 +18,7 @@
     assume NWU (otherwise cob is below cog?).
     -->
-    <xacro:property name="cob" value="0.0 0.0 0.3"/>
+    <xacro:property name="cob" value="0.0 0.0 0.01"/>
     <!-- Volume, see p.31 in Berg2012 -->
-    <xacro:property name="volume" value="1.83826"/>
+    <xacro:property name="volume" value="0.83826"/>
     <xacro:macro name="rexrov_hydro_model" params="namespace">
         <link name="${namespace}/base_link">
@@ -26,7 +26,7 @@
             <volume>${volume}</volume>
             <box>
-                <width>1.5</width>
-                <length>2.6</length>
-                <height>1.6</height>
+                <width>0.3</width>
+                <length>0.62</length>
+                <height>0.47305</height>
             </box>
             <center_of_buoyancy>${cob}</center_of_buoyancy>
@@ -35,18 +35,26 @@
                 <!-- Added mass: see p.28 in Berg2012 -->
                 <added_mass>
-                     779.79 -6.8773 -103.32  8.5426 -165.54 -7.8033
-                    -6.8773    1222   51.29  409.44 -5.8488  62.726
-                    -103.32   51.29  3659.9  6.1112 -386.42  10.774
-                     8.5426  409.44  6.1112   534.9 -10.027  21.019
-                    -165.54 -5.8488 -386.42 -10.027  842.69 -1.1162
-                    -7.8033  62.726  10.775  21.019 -1.1162  224.32
+                    16.93       0.0         0.0         0.0         0.0         0.0
+                    0.0         16.93       0.0         0.0         0.0         0.0
+                    0.0         0.0         16.93       0.0         0.0         0.0
+                    0.0         0.0         0.0         0.0156   0.0014   0.0004
+                    0.0         0.0         0.0         0.0014    0.03      0.0011
+                    0.0         0.0         0.0         0.0004    0.0011  0.0166
                 </added_mass>
-                <!-- Linear damping: see p.31 in Berg2012 -->
                 <linear_damping>
-                    -74.82 -69.48 -728.4 -268.8 -309.77 -105
+                    0.0125   0.0         0.0         0.0         0.0         0.0
+                    0.0         0.0125   0.0         0.0         0.0         0.0
+                    0.0         0.0         0.0499   0.0         0.0         0.0
+                    0.0         0.0         0.0         0.0125   0.0         0.0
+                    0.0         0.0         0.0         0.0         0.0125   0.0
+                    0.0         0.0         0.0         0.0         0.0         0.0499
                 </linear_damping>
-                <!-- Non-linear damping: see p.30 in Berg2012 -->
                 <quadratic_damping>
-                    -748.22 -992.53 -1821.01 -672 -774.44 -523.27
+                    0.0125   0.0         0.0         0.0         0.0         0.0
+                    0.0         0.0125   0.0         0.0         0.0         0.0
+                    0.0         0.0         0.0499   0.0         0.0         0.0
+                    0.0         0.0         0.0         0.0125   0.0         0.0
+                    0.0         0.0         0.0         0.0         0.0125   0.0
+                    0.0         0.0         0.0         0.0         0.0         0.0499
                 </quadratic_damping>
             </hydrodynamic_model>

File: haubentaucher_description/urdf/rexrov_actuators.xacro (robot description, xacro)
@@ -27,11 +27,11 @@
   </xacro:macro>
   <xacro:thruster_macro namespace="${namespace}" thruster_id="0">
-    <origin xyz="0.12 0 0" rpy="0 0 0"/>
+    <origin xyz="0.12 0 -0.1" rpy="-3.14 0 0"/>
   </xacro:thruster_macro>
   <xacro:thruster_macro namespace="${namespace}" thruster_id="1">
-    <origin xyz="0 -0.3 0" rpy="0 0 0"/>
+    <origin xyz="0 -0.205500 0.088000" rpy="0 -1.5707 0"/>
   </xacro:thruster_macro>
   <xacro:thruster_macro namespace="${namespace}" thruster_id="2">
-    <origin xyz="0 0.3 0" rpy="0 0 0"/>
+    <origin xyz="0 0.205500 0.088000" rpy="0 -1.5707 0"/>
   </xacro:thruster_macro>
 </robot>

Commit message: aa

File: haubentaucher_description/urdf/rexrov.gazebo.xacro (robot description, xacro)
@@ -20,5 +20,5 @@
     <xacro:property name="cob" value="0.0 0.0 0.01"/>
     <!-- Volume, see p.31 in Berg2012 -->
-    <xacro:property name="volume" value="0.83826"/>
+    <xacro:property name="volume" value="0.01"/>
     <xacro:macro name="rexrov_hydro_model" params="namespace">
         <link name="${namespace}/base_link">
@@ -35,7 +35,7 @@
                 <!-- Added mass: see p.28 in Berg2012 -->
                 <added_mass>
-                    16.93       0.0         0.0         0.0         0.0         0.0
-                    0.0         16.93       0.0         0.0         0.0         0.0
-                    0.0         0.0         16.93       0.0         0.0         0.0
+                    0.093       0.0         0.0         0.0         0.0         0.0
+                    0.0         0.093       0.0         0.0         0.0         0.0
+                    0.0         0.0         0.093       0.0         0.0         0.0
                     0.0         0.0         0.0         0.0156   0.0014   0.0004
                     0.0         0.0         0.0         0.0014    0.03      0.0011
