Commit message: Addded sensors.

File: haubentaucher_description/urdf/haubentaucher.urdf.xacro (robot description, xacro)
@@ -8,4 +8,5 @@
     <!-- Instantiate kopterworx mechanics "mechanics" -->
     <xacro:include filename="$(find haubentaucher_description)/urdf/haubentaucher_base.urdf.xacro" />
+    <xacro:include filename="$(find haubentaucher_description)/urdf/haubentaucher_sensors.urdf.xacro" />
     <xacro:include filename="$(find rotors_description)/urdf/component_snippets.xacro" />
     <gazebo>
@@ -56,4 +57,31 @@
     <xacro:default_imu namespace="${namespace}" parent_link="${namespace}/base_link" />
     <xacro:ground_truth_imu_and_odometry namespace="${namespace}" parent_link="${namespace}/base_link" />-->
+    <joint name="scan_joint" type="fixed">
+      <parent link="${namespace}/base_link"/>
+      <child link="base_scan"/>
+      <origin xyz="0.0 0 0.05" rpy="0 0 0"/>
+    </joint>
+    <link name="base_scan">
+      <visual>
+        <origin xyz="0 0 0.0" rpy="0 0 0"/>
+        <geometry>
+          <mesh filename="package://hydrone_aerial_underwater_description/meshes/lds.stl" scale="0.001 0.001 0.001"/>
+        </geometry>
+        <material name="dark"/>
+      </visual>
+      <collision>
+        <origin xyz="0.015 0 -0.0065" rpy="0 0 0"/>
+        <geometry>
+          <cylinder length="0.0315" radius="0.055"/>
+        </geometry>
+      </collision>
+      <inertial>
+        <mass value="0.114" />
+        <origin xyz="0 0 0" />
+        <inertia ixx="0.001" ixy="0.0" ixz="0.0"
+                iyy="0.001" iyz="0.0"
+                izz="0.001" />
+      </inertial>
+    </link>
     <!-- Set up hydrodynamic plugin given as input parameter
     <xacro:insert_block name="gazebo"/>-->

Commit message: Addded sensors.

File: haubentaucher_description/urdf/haubentaucher.urdf.xacro (robot description, xacro)
@@ -84,4 +84,11 @@
       </inertial>
     </link>
+    <joint name="camera_joint" type="fixed">
+      <parent link="${namespace}/base_link"/>
+      <child link="camera_link"/>
+      <origin xyz="0.1 0 0.0" rpy="0 0 0"/>
+    </joint>
+    <link name="camera_link">
+    </link>
     <!-- Set up hydrodynamic plugin given as input parameter
     <xacro:insert_block name="gazebo"/>-->

File: haubentaucher_description/urdf/haubentaucher_sensors.urdf.xacro (robot description, xacro)
@@ -43,13 +43,13 @@
         </sensor>
     </gazebo>
-    <gazebo reference="${namespace}/base_link">
+    <gazebo reference="camera_link">
     <sensor type="depth" name="kinect">
-      <pose>0 0 -0.1 0 0 0</pose>
+      <pose>0 0 0 0 0 0</pose>
       <update_rate>30.0</update_rate>
       <camera>
         <horizontal_fov>1.3962634</horizontal_fov>
         <image>
-          <width>100</width>
-          <height>100</height>
+          <width>1280</width>
+          <height>720</height>
           <format>R8G8B8</format>
         </image>
@@ -79,5 +79,5 @@
           <depthImageCameraInfoTopicName>/haubentaucher/camera/depth/camera_info</depthImageCameraInfoTopicName>
           <pointCloudTopicName>/haubentaucher/camera/depth/points</pointCloudTopicName>
-          <frameName>camera_depth_link</frameName>
+          <frameName>camera_link</frameName>
           <pointCloudCutoff>0.5</pointCloudCutoff>
           <pointCloudCutoffMax>3.0</pointCloudCutoffMax>

Commit message: Underwater working.

File: haubentaucher_description/urdf/haubentaucher.urdf.xacro (robot description, xacro)
@@ -3,10 +3,36 @@
     <xacro:property name="namespace" value="haubentaucher" />
     <xacro:property name="max_range" value="8.0"/>
+    <xacro:arg name="inertial_reference_frame" default="world"/>
+    <xacro:arg name="debug" default="0"/>
     <!-- Collision bitmask - By default collides with everything -->
     <xacro:arg name="collision_bitmask" default="-1" />
     <xacro:property name="collision_bitmask" value="$(arg collision_bitmask)" />
+    <xacro:include filename="$(find uuv_descriptions)/urdf/common.urdf.xacro"/>
+    <xacro:include filename="$(find uuv_sensor_ros_plugins)/urdf/sensor_snippets.xacro"/>
+    <xacro:include filename="$(find uuv_gazebo_ros_plugins)/urdf/snippets.xacro"/>
     <!-- Instantiate kopterworx mechanics "mechanics" -->
     <xacro:include filename="$(find haubentaucher_description)/urdf/haubentaucher_base.urdf.xacro" />
+    <xacro:include filename="$(find haubentaucher_description)/urdf/haubentaucher_sensors.urdf.xacro" />
     <xacro:include filename="$(find rotors_description)/urdf/component_snippets.xacro" />
+    <!--<xacro:include filename="$(find haubentaucher_description)/urdf/haubentaucher_actuators.xacro"/>-->
+    <xacro:include filename="$(find haubentaucher_description)/urdf/haubentaucher.gazebo.xacro"/>
+    <!-- Create the rexrov -->
+    <xacro:haubentaucher_base
+        namespace="$(arg namespace)"
+        inertial_reference_frame="$(arg inertial_reference_frame)">
+        <!-- The underwater object plugin is given as an input block parameter to
+         allow the addition of external models of manipulator units -->
+        <gazebo>
+            <plugin name="uuv_plugin" filename="libuuv_underwater_object_ros_plugin.so">
+                <fluid_density>1028.0</fluid_density>
+                <flow_velocity_topic>hydrodynamics/current_velocity</flow_velocity_topic>
+                <debug>$(arg debug)</debug>
+                <!-- Adding the hydrodynamic and hydrostatic parameters for the vehicle-->
+                <xacro:haubentaucher_hydro_model namespace="$(arg namespace)"/>
+            </plugin>
+        </gazebo>
+    </xacro:haubentaucher_base>
+    <!-- Joint state publisher plugin -->
+    <xacro:default_joint_state_publisher namespace="$(arg namespace)" update_rate="50"/>
     <gazebo>
         <plugin name="gazebo_ros_control" filename="libgazebo_ros_control.so">
@@ -56,4 +82,38 @@
     <xacro:default_imu namespace="${namespace}" parent_link="${namespace}/base_link" />
     <xacro:ground_truth_imu_and_odometry namespace="${namespace}" parent_link="${namespace}/base_link" />-->
+    <joint name="scan_joint" type="fixed">
+      <parent link="${namespace}/base_link"/>
+      <child link="base_scan"/>
+      <origin xyz="0.0 0 0.05" rpy="0 0 0"/>
+    </joint>
+    <link name="base_scan">
+      <visual>
+        <origin xyz="0 0 0.0" rpy="0 0 0"/>
+        <geometry>
+          <mesh filename="package://hydrone_aerial_underwater_description/meshes/lds.stl" scale="0.001 0.001 0.001"/>
+        </geometry>
+        <material name="dark"/>
+      </visual>
+      <collision>
+        <origin xyz="0.015 0 -0.0065" rpy="0 0 0"/>
+        <geometry>
+          <cylinder length="0.0315" radius="0.055"/>
+        </geometry>
+      </collision>
+      <inertial>
+        <mass value="0.114" />
+        <origin xyz="0 0 0" />
+        <inertia ixx="0.001" ixy="0.0" ixz="0.0"
+                iyy="0.001" iyz="0.0"
+                izz="0.001" />
+      </inertial>
+    </link>
+    <joint name="camera_joint" type="fixed">
+      <parent link="${namespace}/base_link"/>
+      <child link="camera_link"/>
+      <origin xyz="0.1 0 0.0" rpy="0 0 0"/>
+    </joint>
+    <link name="camera_link">
+    </link>
     <!-- Set up hydrodynamic plugin given as input parameter
     <xacro:insert_block name="gazebo"/>-->

File: haubentaucher_description/urdf/haubentaucher_base.urdf.xacro (robot description, xacro)
@@ -38,4 +38,22 @@
         <inertia ixx="0.02953" ixy="0.0001" ixz="-0.0142" iyy="0.2303" iyz="0.0038" izz="0.1604" />  <!-- updated 15.09.2023 -->
     </xacro:property>
+    <xacro:macro name="haubentaucher_base" params="namespace *gazebo inertial_reference_frame">
+        <!-- base_link according to ROS conventions: x forward, z up
+        <link name="${namespace}/base_link">
+          <inertial>
+            <mass value="${mass}"/>
+            <origin xyz="0 0 0"/>
+            <inertia ixx="0.02953" ixy="0.0001" ixz="-0.0142" iyy="0.2303" iyz="0.0038" izz="0.1604" />
+        </link>-->
+        <!-- Set up hydrodynamic plugin given as input parameter -->
+        <xacro:insert_block name="gazebo"/>
+        <!-- optional: plugin to test compare Gazebo's returned accelerations
+        <gazebo>
+          <plugin name="${namespace}_test_plugin" filename="libuuv_accelerations_test_plugin.so">
+            <link_name>${namespace}/base_link</link_name>
+          </plugin>
+        </gazebo> -->
+        <xacro:include filename="$(find haubentaucher_description)/urdf/haubentaucher_actuators.xacro"/>
+    </xacro:macro>
     <!-- inertia of a single rotor, assuming it is a cuboid. Height=3mm, width=15mm -->
     <xacro:property name="rotor_inertia">
@@ -60,6 +78,6 @@
   <xacro:vertical_rotor
     robot_namespace="${namespace}"
-    suffix="front"
-    direction="cw"
+    suffix="front_right"
+    direction="ccw"
     motor_constant="${motor_constant}"
     moment_constant="${moment_constant}"
@@ -73,13 +91,13 @@
     rotor_drag_coefficient="${rotor_drag_coefficient}"
     rolling_moment_coefficient="${rolling_moment_coefficient}"
-    color="Red"
+    color="Blue"
     use_own_mesh="false"
     mesh="">
-    <origin xyz="${rotor_x_offset} ${rotor_y_offset} ${rotor_offset_top}" rpy="0 0 0" /> <!-- look at the definition above to understand how the position is defined -->
+    <origin xyz="${rotor_x_offset} -${rotor_y_offset} ${rotor_offset_top}" rpy="0 0 0" /> <!-- look at the definition above to understand how the position is defined -->
     <xacro:insert_block name="rotor_inertia" />
   </xacro:vertical_rotor>
   <xacro:vertical_rotor
     robot_namespace="${namespace}"
-    suffix="left"
+    suffix="back_left"
     direction="ccw"
     motor_constant="${motor_constant}"
@@ -97,10 +115,10 @@
     use_own_mesh="false"
     mesh="">
-    <origin xyz="${rotor_x_offset} -${rotor_y_offset} ${rotor_offset_top}" rpy="0 0 0" />
+    <origin xyz="-${rotor_x_offset} ${rotor_y_offset} ${rotor_offset_top}" rpy="0 0 0" />
     <xacro:insert_block name="rotor_inertia" />
   </xacro:vertical_rotor>
   <xacro:vertical_rotor
     robot_namespace="${namespace}"
-    suffix="back"
+    suffix="front_left"
     direction="cw"
     motor_constant="${motor_constant}"
@@ -115,14 +133,14 @@
     rotor_drag_coefficient="${rotor_drag_coefficient}"
     rolling_moment_coefficient="${rolling_moment_coefficient}"
-    color="Blue"
+    color="Red"
     use_own_mesh="false"
     mesh="">
-    <origin xyz="-${rotor_x_offset} ${rotor_y_offset} ${rotor_offset_top}" rpy="0 0 0" />
+    <origin xyz="${rotor_x_offset} ${rotor_y_offset} ${rotor_offset_top}" rpy="0 0 0" />
     <xacro:insert_block name="rotor_inertia" />
   </xacro:vertical_rotor>
   <xacro:vertical_rotor
     robot_namespace="${namespace}"
-    suffix="right"
-    direction="ccw"
+    suffix="back_right"
+    direction="cw"
     motor_constant="${motor_constant}"
     moment_constant="${moment_constant}"
@@ -136,5 +154,5 @@
     rotor_drag_coefficient="${rotor_drag_coefficient}"
     rolling_moment_coefficient="${rolling_moment_coefficient}"
-    color="Blue"
+    color="Red"
     use_own_mesh="false"
     mesh="">

File: haubentaucher_description/urdf/haubentaucher_multirotor_base.xacro (robot description, xacro)
@@ -17,44 +17,4 @@
 -->
 <robot xmlns:xacro="http://ros.org/wiki/xacro">
-  <!--
-  Center of buoyancy according to eq. (3.1) p. 28 in Berg2012.
-  The original values, [0.0822, -0.00773, 0.3872] however, seem to
-  assume NWU (otherwise cob is below cog?).
-  -->
-  <xacro:property name="cob" value="0.0 0.0 0.3"/>
-  <!-- Volume, see p.31 in Berg2012 -->
-  <xacro:property name="volume" value="0.83826"/>
-  <xacro:macro name="rexrov_hydro_model" params="namespace">
-      <link name="${namespace}/base_link_inertia">
-          <neutrally_buoyant>1</neutrally_buoyant>
-          <volume>${volume}</volume>
-          <box>
-              <width>1.5</width>
-              <length>2.6</length>
-              <height>1.6</height>
-          </box>
-          <center_of_buoyancy>${cob}</center_of_buoyancy>
-          <hydrodynamic_model>
-              <type>fossen</type>
-              <!-- Added mass: see p.28 in Berg2012 -->
-              <added_mass>
-                   779.79 -6.8773 -103.32  8.5426 -165.54 -7.8033
-                  -6.8773    1222   51.29  409.44 -5.8488  62.726
-                  -103.32   51.29  3659.9  6.1112 -386.42  10.774
-                   8.5426  409.44  6.1112   534.9 -10.027  21.019
-                  -165.54 -5.8488 -386.42 -10.027  842.69 -1.1162
-                  -7.8033  62.726  10.775  21.019 -1.1162  224.32
-              </added_mass>
-              <!-- Linear damping: see p.31 in Berg2012 -->
-              <linear_damping>
-                  -74.82 -69.48 -728.4 -268.8 -309.77 -105
-              </linear_damping>
-              <!-- Non-linear damping: see p.30 in Berg2012 -->
-              <quadratic_damping>
-                  -748.22 -992.53 -1821.01 -672 -774.44 -523.27
-              </quadratic_damping>
-          </hydrodynamic_model>
-      </link>
-  </xacro:macro>
   <!-- Macro for the inertia of a box -->
   <xacro:macro name="box_inertia" params="x y z mass">
@@ -112,13 +72,4 @@
         <linkName>${robot_namespace}/base_link</linkName>
         <rotorVelocitySlowdownSim>${rotor_velocity_slowdown_sim}</rotorVelocitySlowdownSim>
-      </plugin>
-    </gazebo>
-    <gazebo>
-      <plugin name="uuv_plugin" filename="libuuv_underwater_object_ros_plugin.so">
-        <fluid_density>1028.0</fluid_density>
-        <flow_velocity_topic>hydrodynamics/current_velocity</flow_velocity_topic>
-        <debug>True</debug>
-        <!-- Adding the hydrodynamic and hydrostatic parameters for the vehicle-->
-        <xacro:rexrov_hydro_model namespace="${robot_namespace}"/>
       </plugin>
     </gazebo>

Commit message: a

File: haubentaucher_description/urdf/haubentaucher.urdf.xacro (robot description, xacro)
@@ -116,7 +116,3 @@
     <link name="camera_link">
     </link>
-    <!-- Set up hydrodynamic plugin given as input parameter
-    <xacro:insert_block name="gazebo"/>-->
-    <!-- <xacro:include filename="$(find hydrone_aerial_underwater_description)/urdf/hydrone_aerial_underwater_sensors.xacro" /> -->
-    <!-- <xacro:include filename="$(find hydrone_aerial_underwater_description)/urdf/hydrone_aerial_underwater_actuators.xacro" /> -->
 </robot>

File: haubentaucher_description/urdf/haubentaucher_actuators.xacro (robot description, xacro)
@@ -16,5 +16,5 @@
   <!-- Thruster joint and link snippet -->
   <xacro:macro name="thruster_macro"
-    params="namespace thruster_id *origin">
+    params="namespace thruster_id *origin *axis">
     <xacro:thruster_module_first_order_basic_fcn_macro
       namespace="${namespace}"
@@ -24,14 +24,18 @@
       rotor_constant="0.00031">
       <xacro:insert_block name="origin"/>
+      <xacro:insert_block name="axis"/>
     </xacro:thruster_module_first_order_basic_fcn_macro>
   </xacro:macro>
   <xacro:thruster_macro namespace="${namespace}" thruster_id="0">
-    <origin xyz="0.12 0 -0.1" rpy="-3.14 0 0"/>
+    <origin xyz="0.12 0 -0.1" rpy="${pi} 0 0"/>
+    <axis xyz="0 0 1"/>
   </xacro:thruster_macro>
   <xacro:thruster_macro namespace="${namespace}" thruster_id="1">
-    <origin xyz="0 -0.205500 0.088000" rpy="0 -1.5707 0"/>
+    <origin xyz="0 -0.205500 0.088000" rpy="0 ${pi/2} 0"/>
+    <axis xyz="0 0 1"/>
   </xacro:thruster_macro>
   <xacro:thruster_macro namespace="${namespace}" thruster_id="2">
-    <origin xyz="0 0.205500 0.088000" rpy="0 -1.5707 0"/>
+    <origin xyz="0 0.205500 0.088000" rpy="0 ${pi/2} 0"/>
+    <axis xyz="0 0 1"/>
   </xacro:thruster_macro>
 </robot>

File: haubentaucher_description/urdf/haubentaucher_sensors.urdf.xacro (robot description, xacro)
@@ -95,3 +95,89 @@
     </sensor>
   </gazebo>
+  <xacro:macro name="multibosta_sonar"
+    params="namespace suffix parent_link topic mass update_rate
+      samples fov range_min range_max range_stddev mesh
+      *inertia *origin *visual">
+    <!-- Sensor link -->
+    <link name="${namespace}/sonar${suffix}_link">
+      <inertial>
+        <xacro:insert_block name="inertia" />
+        <mass value="${mass}" />
+        <origin xyz="0 0 0" rpy="0 0 0" />
+      </inertial>
+      <xacro:insert_block name="visual" />
+      <xacro:no_collision/>
+    </link>
+  <joint name="${namespace}_sonar${suffix}_joint" type="revolute">
+    <xacro:insert_block name="origin" />
+    <parent link="${parent_link}" />
+    <child link="${namespace}/sonar${suffix}_link" />
+    <limit upper="0" lower="0" effort="0" velocity="0" />
+    <axis xyz="1 0 0"/>
+  </joint>
+  <gazebo reference="${namespace}/sonar${suffix}_link">
+    <sensor type="ray" name="sonar${suffix}">
+      <pose>0 0 0 0 0 0</pose>
+      <visualize>false</visualize>
+      <update_rate>${update_rate}</update_rate>
+      <ray>
+        <scan>
+          <horizontal>
+            <samples>${samples}</samples>
+            <resolution>1</resolution>
+            <min_angle>-${0.5*fov}</min_angle>
+            <max_angle>${0.5*fov}</max_angle>
+          </horizontal>
+        </scan>
+        <range>
+          <min>${range_min}</min>
+          <max>${range_max}</max>
+          <resolution>0.01</resolution>
+        </range>
+        <noise>
+          <type>gaussian</type>
+          <mean>0.0</mean>
+          <stddev>${range_stddev}</stddev>
+        </noise>
+      </ray>
+      <plugin name="sonar${suffix}_controller" filename="libgazebo_ros_gpu_laser.so">
+        <topicName>${topic}</topicName>
+        <frameName>sonar${suffix}_link</frameName>
+      </plugin>
+      <!-- TODO: Separate switchable sonar version in another macro -->
+      <!-- <plugin name="switchable_sonar{suffix}_ros_interface" filename="libuuv_gazebo_ros_switchable_gpu_ray_sensor.so">
+          <namespace>${namespace}</namespace>
+          <input_topic>${topic}</input_topic>
+      </plugin> -->
+    </sensor>
+  </gazebo>
+  </xacro:macro>
+  <xacro:macro name="sonar_bosta" params="namespace parent_link *origin">
+    <xacro:multibosta_sonar
+      namespace="${namespace}"
+      suffix=""
+      parent_link="${parent_link}"
+      topic="sonar"
+      mass="0.02"
+      update_rate="500"
+      samples="20"
+      fov="1.5708"
+      range_min="1.0"
+      range_max="8.0"
+      range_stddev="0.027"
+      mesh="">
+      <inertia ixx="0.00001" ixy="0.0" ixz="0.0" iyy="0.00001" iyz="0.0" izz="0.00001" />
+      <xacro:insert_block name="origin" />
+      <visual>
+        <origin xyz="0 0 0" rpy="${-pi/2} 0 0"/>
+        <geometry>
+          <mesh filename="file://$(find haubentaucher_description)/meshes/ping360.stl" scale="0.00001 0.00001 0.00001"/>
+        </geometry>
+      </visual>
+    </xacro:multibosta_sonar>
+  </xacro:macro>
+  <!-- Forward-looking sonar sensor -->
+  <xacro:sonar_bosta namespace="${namespace}" parent_link="${namespace}/base_link">
+    <origin xyz="0 0 -0.16" rpy="0 0 0"/>
+  </xacro:sonar_bosta>
 </robot>
