Commit message: Underwater actuators working.

File: haubentaucher_description/urdf/haubentaucher.gazebo.xacro (robot description, xacro)
@@ -33,5 +33,5 @@
             <hydrodynamic_model>
                 <type>fossen</type>
-                <!-- Added mass: see p.28 in Berg2012 -->
+                <!--Added mass: see p.28 in Berg2012
                 <added_mass>
                     0.093       0.0         0.0         0.0         0.0         0.0
@@ -41,6 +41,14 @@
                     0.0         0.0         0.0         0.0014    0.03      0.0011
                     0.0         0.0         0.0         0.0004    0.0011  0.0166
-                </added_mass>
-                <linear_damping>
+                </added_mass>-->
+                 <added_mass>
+                     1.7182 0 0 0 0 0
+                     0 0 0 0 0 0
+                     0 0 2.468 0 0 0
+                     0 0 0 0 0 0
+                     0 0 0 0 1.2481 0
+                     0 0 0 0 0 1.4006
+                 </added_mass>
+                <!--<linear_damping>
                     0.0125   0.0         0.0         0.0         0.0         0.0
                     0.0         0.0125   0.0         0.0         0.0         0.0
@@ -49,6 +57,9 @@
                     0.0         0.0         0.0         0.0         0.0125   0.0
                     0.0         0.0         0.0         0.0         0.0         0.0499
+                </linear_damping>-->
+                <linear_damping>
+                    -11.7391 -20 -31.8678 -25 -44.9085 -5
                 </linear_damping>
-                <quadratic_damping>
+                <!--<quadratic_damping>
                     0.0125   0.0         0.0         0.0         0.0         0.0
                     0.0         0.0125   0.0         0.0         0.0         0.0
@@ -57,4 +68,7 @@
                     0.0         0.0         0.0         0.0         0.0125   0.0
                     0.0         0.0         0.0         0.0         0.0         0.0499
+                </quadratic_damping>-->
+                <quadratic_damping>
+                    0 0 0 0 0 0
                 </quadratic_damping>
             </hydrodynamic_model>

File: haubentaucher_description/urdf/haubentaucher.urdf.xacro (robot description, xacro)
@@ -89,5 +89,5 @@
     <link name="base_scan">
       <visual>
-        <origin xyz="0 0 0.0" rpy="0 0 0"/>
+        <origin xyz="0 0 0.005" rpy="0 ${pi} 0"/>
         <geometry>
           <mesh filename="package://hydrone_aerial_underwater_description/meshes/lds.stl" scale="0.001 0.001 0.001"/>

File: haubentaucher_description/urdf/haubentaucher_actuators.xacro (robot description, xacro)
@@ -22,5 +22,5 @@
       mesh_filename="${prop_mesh_file}"
       dyn_time_constant="0.05"
-      rotor_constant="0.00031">
+      rotor_constant="0.001">
       <xacro:insert_block name="origin"/>
       <xacro:insert_block name="axis"/>
@@ -28,13 +28,13 @@
   </xacro:macro>
   <xacro:thruster_macro namespace="${namespace}" thruster_id="0">
-    <origin xyz="0.12 0 -0.1" rpy="${pi} 0 0"/>
+    <origin xyz="0.12 0.0005 -0.1" rpy="${pi} 0 0"/>
     <axis xyz="0 0 1"/>
   </xacro:thruster_macro>
   <xacro:thruster_macro namespace="${namespace}" thruster_id="1">
-    <origin xyz="0 -0.205500 0.088000" rpy="0 ${pi/2} 0"/>
+    <origin xyz="-0.025 -0.205500 0.08500" rpy="0 ${pi/2} 0"/>
     <axis xyz="0 0 1"/>
   </xacro:thruster_macro>
   <xacro:thruster_macro namespace="${namespace}" thruster_id="2">
-    <origin xyz="0 0.205500 0.088000" rpy="0 ${pi/2} 0"/>
+    <origin xyz="-0.025 0.205500 0.08500" rpy="0 ${pi/2} 0"/>
     <axis xyz="0 0 1"/>
   </xacro:thruster_macro>

File: haubentaucher_description/urdf/haubentaucher_sensors.urdf.xacro (robot description, xacro)
@@ -13,5 +13,5 @@
         <sensor type="ray" name="VLP-16-VLP16-Simplified">
         <pose>0 0 0 0 0 0</pose>
-        <visualize>false</visualize>
+        <visualize>true</visualize>
         <update_rate>500</update_rate>
         <ray>
@@ -119,5 +119,5 @@
     <sensor type="ray" name="sonar${suffix}">
       <pose>0 0 0 0 0 0</pose>
-      <visualize>false</visualize>
+      <visualize>true</visualize>
       <update_rate>${update_rate}</update_rate>
       <ray>
